Commit message: Agregue los limites a las juntas 2,3 y 5, tambien agregue un sistema que regresa todo a cero y un pequeño sistema para ver las coordenadas rectangulares, el cero es angular

File: src/assets/models/robot_fanuc.urdf (robot description, URDF)
Before this commit: robot fanuc_m900ia260l, 12 links, 11 joints
Joints:
- joint joint_2: limit lower=-1.308997 upper=1.308997 effort=0 velocity=1.832596 -> lower=-1.4 upper=1.76 effort=0 velocity=1.832596
- joint joint_3: limit lower=-2.116665 upper=1.570796 effort=0 velocity=1.658063 -> lower=-1.23 upper=1.76 effort=0 velocity=1.658063
- joint joint_5: limit lower=-2.181662 upper=2.181662 effort=0 velocity=2.094395 -> lower=-1.76 upper=1.92 effort=0 velocity=2.094395
